Commit message: Add files via upload

File: seguidor/robot_bruno/kinetic.xacro (robot description, xacro)
@@ -2,5 +2,5 @@
 <robot xmlns:xacro="http://www.ros.org/wiki/xacro" >
   <joint name="kinetic_joint" type="fixed">
-    <origin xyz="${tamanho_x/2} 0 0" rpy="0.0 0.0 0.0"/>
+    <origin xyz="${tamanho_x/2} 0 0.2" rpy="0.0 45.0 0.0"/>
     <parent link="corpo_link"/>
     <child link="kinetic_link"/>
@@ -9,5 +9,5 @@
     <visual>
       <material name="white"/>
-      <origin xyz="0.0 0.0 0.0" rpy="${pi} 0.0 0.0"/>
+      <origin xyz="0.0 0.0 0.2" rpy="${pi} 45.0 0.0"/>
       <geometry>
         <box size="0.05 0.05 0.05"/>
@@ -18,5 +18,5 @@
         <parent link="kinetic_link"/>
         <child link="dumb_kinetic"/>
-        <origin xyz="0 0 0" rpy="${-pi/2} 0 ${-pi/2}"/>
+        <origin xyz="0 0 0.2" rpy="${-pi/2} 45.0 ${-pi/2}"/>
     </joint>
   <link name="dumb_kinetic">

Commit message: Add files via upload

File: seguidor/robot_bruno/kinetic.xacro (robot description, xacro)
@@ -2,5 +2,5 @@
 <robot xmlns:xacro="http://www.ros.org/wiki/xacro" >
   <joint name="kinetic_joint" type="fixed">
-    <origin xyz="${tamanho_x/2} 0 0.2" rpy="0.0 45.0 0.0"/>
+    <origin xyz="${tamanho_x/2} 0 0.08" rpy="0.0 45.0 0.0"/>
     <parent link="corpo_link"/>
     <child link="kinetic_link"/>
@@ -9,5 +9,5 @@
     <visual>
       <material name="white"/>
-      <origin xyz="0.0 0.0 0.2" rpy="${pi} 45.0 0.0"/>
+      <origin xyz="0.0 0.0 0.08" rpy="${pi} 45.0 0.0"/>
       <geometry>
         <box size="0.05 0.05 0.05"/>
@@ -18,5 +18,5 @@
         <parent link="kinetic_link"/>
         <child link="dumb_kinetic"/>
-        <origin xyz="0 0 0.2" rpy="${-pi/2} 45.0 ${-pi/2}"/>
+        <origin xyz="0 0 0.08" rpy="${-pi/2} 45.0 ${-pi/2}"/>
     </joint>
   <link name="dumb_kinetic">
